File: esp-jtag.sch (KiCad schematic (older format))
At the start: 70 parts, among them J1 USB_B_Micro, J2 JTAG, Q1 WST03P06, Q2 S8050, Q3 S8050, SW1 SW_SPST, SW2 SW_SPST, U1 74AHC1GU04, U2 SN74AHC125RGY, U3 AMS1117-3.3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

Commit message: Layout and route the PCB
Prepare the PCB layout by arranging the components
Route all traces and rectify mistakes in the connections
Add ground pours on top and bottom copper
Update the preview images and the README file
Parts:
- added L1: karibe_logo, artwork:karibe_logo, symbol myRF:karibe_logo
- J2: LCSC # C12650 -> (none); Mfr # C12650 -> (none)
Connections:
- net ESP_TCK: now also J2.4 (Pin_4)
- net ESP_TDI: now also J2.8 (Pin_8)
- net ESP_TDO: now also J2.6 (Pin_6)
- net ESP_TMS: now also J2.2 (Pin_2)
- net FT_RxD: now also J2.7 (Pin_7); no longer J2.5 (Pin_5)
- net FT_TCK: no longer J2.4 (Pin_4)
- net FT_TDI: no longer J2.8 (Pin_8)
- net FT_TDO: no longer J2.6 (Pin_6)
- net FT_TMS: no longer J2.2 (Pin_2)
- net FT_TxD: now also J2.5 (Pin_5); no longer J2.7 (Pin_7)
- net GND: now also J2.10 (Pin_10)
Changed lines of the file:
@@
 	2150 7200 2300 7200
-$Comp
-L Regulator_Linear:AMS1117-3.3 U3
-U 1 1 5DE54B69
-P 4300 4800
-F 0 "U3" H 4300 5042 50  0000 C CNN
-F 1 "AMS1117-3.3" H 4300 4951 50  0000 C CNN
-F 2 "Package_TO_SOT_SMD:SOT-223-3_TabPin2" H 4300 5000 50  0001 C CNN
-F 3 "http://www.advanced-monolithic.com/pdf/ds1117.pdf" H 4400 4550 50  0001 C CNN
-F 4 "AMS1117-3.3" H 4300 4800 50  0001 C CNN "Mfr #"
-F 5 "C6186" H 4300 4800 50  0001 C CNN "LCSC #"
-	1    4300 4800
-	1    0    0    -1
-$EndComp
 $Comp
 L Device:C_Small C5
@@
 	7800 800  7800 1650
 Connection ~ 7000 800
-$Comp
-L Connector_Generic:Conn_02x05_Odd_Even J2
-U 1 1 5E2C9CB5
-P 1850 5250
-F 0 "J2" H 1900 5667 50  0000 C CNN
-F 1 "JTAG" H 1900 5576 50  0000 C CNN
-F 2 "Connector_PinHeader_1.27mm:PinHeader_2x05_P1.27mm_Vertical_SMD" H 1850 5250 50  0001 C CNN
-F 3 "https://datasheet.lcsc.com/szlcsc/1810221720_Boom-Precision-Elec-C12650_C12650.pdf" H 1850 5250 50  0001 C CNN
-F 4 "C12650" H 1850 5250 50  0001 C CNN "Mfr #"
-F 5 "C12650" H 1850 5250 50  0001 C CNN "LCSC #"
-	1    1850 5250
-	1    0    0    -1
-$EndComp
 Text GLabel 2150 5150 2    50   Input ~ 0
-FT_TCK
+ESP_TCK
 Text GLabel 2150 5350 2    50   Input ~ 0
-FT_TDI
+ESP_TDI
 Text GLabel 2150 5250 2    50   Input ~ 0
-FT_TDO
+ESP_TDO
 Text GLabel 2150 5050 2    50   Input ~ 0
-FT_TMS
-NoConn ~ 2150 5450
+ESP_TMS
 $Comp
 L power:GND #PWR0128
@@
 	1    0    0    -1
 $EndComp
+Text GLabel 1650 5250 0    50   Input ~ 0
+FT_TxD
 Text GLabel 1650 5350 0    50   Input ~ 0
-FT_TxD
-Text GLabel 1650 5250 0    50   Input ~ 0
 FT_RxD
 Wire Wire Line
@@
 Text GLabel 7000 2950 0    50   Input ~ 0
 USB_DM
+$Comp
+L Regulator_Linear:AMS1117-3.3 U3
+U 1 1 5DE54B69
+P 4300 4800
+F 0 "U3" H 4300 5042 50  0000 C CNN
+F 1 "AMS1117-3.3" H 4300 4951 50  0000 C CNN
+F 2 "Package_TO_SOT_SMD:SOT-223-3_TabPin2" H 4300 5000 50  0001 C CNN
+F 3 "http://www.advanced-monolithic.com/pdf/ds1117.pdf" H 4400 4550 50  0001 C CNN
+F 4 "AMS1117-3.3" H 4300 4800 50  0001 C CNN "Mfr #"
+F 5 "C6186" H 4300 4800 50  0001 C CNN "LCSC #"
+	1    4300 4800
+	1    0    0    -1
+$EndComp
+$Comp
+L Connector_Generic:Conn_02x05_Odd_Even J2
+U 1 1 5E2C9CB5
+P 1850 5250
+F 0 "J2" H 1900 5667 50  0000 C CNN
+F 1 "JTAG" H 1900 5576 50  0000 C CNN
+F 2 "Connector_PinHeader_1.27mm:PinHeader_2x05_P1.27mm_Vertical_SMD" H 1850 5250 50  0001 C CNN
+F 3 "~" H 1850 5250 50  0001 C CNN
+	1    1850 5250
+	1    0    0    -1
+$EndComp
+$Comp
+L power:GND #PWR0137
+U 1 1 5DCEA1EC
+P 2150 5450
+F 0 "#PWR0137" H 2150 5200 50  0001 C CNN
+F 1 "GND" H 2155 5277 50  0000 C CNN
+F 2 "" H 2150 5450 50  0001 C CNN
+F 3 "" H 2150 5450 50  0001 C CNN
+	1    2150 5450
+	1    0    0    -1
+$EndComp
+$Comp
+L myRF:karibe_logo L1
+U 1 1 5DD057EE
+P 11000 7000
+F 0 "L1" H 10887 7225 50  0001 C CNN
+F 1 "karibe_logo" H 10887 7133 50  0001 C CNN
+F 2 "artwork:karibe_logo" H 11000 7000 50  0001 C CNN
+F 3 "" H 11000 7000 50  0001 C CNN
+	1    11000 7000
+	1    0    0    -1
+$EndComp
+NoConn ~ 11100 7000
+$Comp
+L Graphic:Logo_Open_Hardware_Small #LOGO1
+U 1 1 5DD4DA49
+P 10300 6900
+F 0 "#LOGO1" H 10300 7175 50  0001 C CNN
+F 1 "Logo_Open_Hardware_Small" H 10300 6675 50  0001 C CNN
+F 2 "" H 10300 6900 50  0001 C CNN
+F 3 "~" H 10300 6900 50  0001 C CNN
+	1    10300 6900
+	1    0    0    -1
+$EndComp
 $EndSCHEMATC

Commit message: Minor tweaks
Finalize PCB layout, especially top silkscreen
Export ray-tracing renders
Update the README file
Parts:
- U5: symbol Interface_USB:FT2232H -> esp-jtag-rescue:FT2232H-Interface_USB
Connections:
- no-connect marks 26 -> 25
Other:
- note added: "TODO:\nAdd 5V torelance using a jumper to choose between VDD and VCC voltages\nGenerate gerber files for manufacturing PCBs"
Changed lines of the file:
@@
 EESchema Schematic File Version 4
-LIBS:esp-jtag-cache
 EELAYER 30 0
 EELAYER END
@@
 $EndComp
 $Comp
-L Interface_USB:FT2232H U5
+L esp-jtag-rescue:FT2232H-Interface_USB U5
 U 1 1 5DE5FE96
 P 8200 3850
@@
 $EndComp
 $Comp
-L myRF:karibe_logo L1
-U 1 1 5DD057EE
-P 11000 7000
-F 0 "L1" H 10887 7225 50  0001 C CNN
-F 1 "karibe_logo" H 10887 7133 50  0001 C CNN
-F 2 "artwork:karibe_logo" H 11000 7000 50  0001 C CNN
-F 3 "" H 11000 7000 50  0001 C CNN
-	1    11000 7000
-	1    0    0    -1
-$EndComp
-NoConn ~ 11100 7000
-$Comp
 L Graphic:Logo_Open_Hardware_Small #LOGO1
 U 1 1 5DD4DA49
@@
 	1    0    0    -1
 $EndComp
+$Comp
+L myRF:karibe_logo L1
+U 1 1 5DC86638
+P 11145 7275
+F 0 "L1" H 11095 7175 50  0001 C CNN
+F 1 "karibe_logo" H 11145 7375 50  0001 C CNN
+F 2 "artwork:karibe_logo" H 11145 7275 50  0001 C CNN
+F 3 "" H 11145 7275 50  0001 C CNN
+	1    11145 7275
+	1    0    0    -1
+$EndComp
+Text Notes 12105 2005 0    50   ~ 0
+TODO:\nAdd 5V torelance using a jumper to choose between VDD and VCC voltages\nGenerate gerber files for manufacturing PCBs
 $EndSCHEMATC
